Commit message: fgseth

File: new_manipulator/urdf/model.urdf (robot description, URDF)
Before this commit: robot new_manipulator, 12 links, 11 joints
Joints:
- joint joint_4: limit lower=-3.14 upper=3.14 effort=0 velocity=0 -> lower=-2.39 upper=0.715 effort=0 velocity=0

Commit message: servoing works

File: new_manipulator/urdf/model.urdf (robot description, URDF)
Before this commit: robot new_manipulator, 12 links, 11 joints
Joints:
- joint base_joint: origin xyz=0.0 0.0 -0.17 rpy=0 0 0 -> xyz=0.0 0.0 0.0 rpy=0 0 0
- joint fake_joint: limit lower=-1.14159 upper=1.14159 effort=0 velocity=0 -> lower=-3.14159 upper=3.14159 effort=0 velocity=0
- joint joint_4: limit lower=-2.39 upper=0.715 effort=0 velocity=0 -> lower=-3.14 upper=3.14 effort=0 velocity=0

File: new_manipulator_moveit_config/config/model.urdf (robot description, URDF)
Before this commit: robot new_manipulator, 12 links, 11 joints
Joints:
- joint fake_joint: limit lower=-1.14159 upper=1.14159 effort=0 velocity=0 -> lower=-3.14159 upper=3.14159 effort=0 velocity=0
- joint joint_4: limit lower=-2.39 upper=0.715 effort=0 velocity=0 -> lower=-3.14 upper=3.14 effort=0 velocity=0
